Commit message: abad 관절 추가, 좌우 모션 추가

File: robot_model.urdf (robot description, URDF)
Before this commit: robot quadruped_robot, 3 links, 2 joints
Links:
- added link abad_link, mass 0.3; collision cylinder length=0.05 radius=0.02; visual cylinder length=0.05 radius=0.02
Joints:
- added joint abad_joint: type revolute, parent base_link, child abad_link, origin xyz=0 -0.095 0 rpy=0 0 0, axis 1 0 0, limit lower=-1.5 upper=1.5 effort=1.0 velocity=1.0
- joint hip_joint: parent base_link -> abad_link

Commit message: 4족보행으로 추가

File: robot_model.urdf (robot description, URDF)
Before this commit: robot quadruped_robot, 4 links, 3 joints
Links:
- removed link abad_link
- removed link hip_link
- removed link knee_link
- added link back_left_abad_link, mass 0.3; visual cylinder length=0.05 radius=0.02
- added link back_left_hip_link, mass 0.5; collision cylinder length=0.3 radius=0.03; visual cylinder length=0.3 radius=0.03
- added link back_left_knee_link, mass 0.3; collision cylinder length=0.3 radius=0.03; visual cylinder length=0.3 radius=0.03
- added link back_right_abad_link, mass 0.3; visual cylinder length=0.05 radius=0.02
- added link back_right_hip_link, mass 0.5; collision cylinder length=0.3 radius=0.03; visual cylinder length=0.3 radius=0.03
- added link back_right_knee_link, mass 0.3; collision cylinder length=0.3 radius=0.03; visual cylinder length=0.3 radius=0.03
- added link front_left_abad_link, mass 0.3; visual cylinder length=0.05 radius=0.02
- added link front_left_hip_link, mass 0.5; collision cylinder length=0.3 radius=0.03; visual cylinder length=0.3 radius=0.03
- added link front_left_knee_link, mass 0.3; collision cylinder length=0.3 radius=0.03; visual cylinder length=0.3 radius=0.03
- added link front_right_abad_link, mass 0.3; visual cylinder length=0.05 radius=0.02
- added link front_right_hip_link, mass 0.5; collision cylinder length=0.3 radius=0.03; visual cylinder length=0.3 radius=0.03
- added link front_right_knee_link, mass 0.3; collision cylinder length=0.3 radius=0.03; visual cylinder length=0.3 radius=0.03
- link base_link: geometry collision box size=0.3 0.3 0.1; visual box size=0.3 0.3 0.1
Joints:
- removed joint abad_joint
- removed joint hip_joint
- removed joint knee_joint
- added joint back_left_abad_joint: type revolute, parent base_link, child back_left_abad_link, origin xyz=-0.1 0.1 0 rpy=0 0 0, axis 1 0 0, limit lower=-1.5 upper=1.5 effort=1.0 velocity=1.0
- added joint back_left_hip_joint: type revolute, parent back_left_abad_link, child back_left_hip_link, origin xyz=0 0.02 0 rpy=0 0 0, axis 0 1 0, limit lower=-3.14 upper=3.14 effort=1.0 velocity=1.0
- added joint back_left_knee_joint: type revolute, parent back_left_hip_link, child back_left_knee_link, origin xyz=0 0.02 -0.3 rpy=0 0 0, axis 0 1 0, limit lower=-3.14 upper=3.14 effort=1.0 velocity=1.0
- added joint back_right_abad_joint: type revolute, parent base_link, child back_right_abad_link, origin xyz=-0.1 -0.1 0 rpy=0 0 0, axis 1 0 0, limit lower=-1.5 upper=1.5 effort=1.0 velocity=1.0
- added joint back_right_hip_joint: type revolute, parent back_right_abad_link, child back_right_hip_link, origin xyz=0 -0.02 0 rpy=0 0 0, axis 0 1 0, limit lower=-3.14 upper=3.14 effort=1.0 velocity=1.0
- added joint back_right_knee_joint: type revolute, parent back_right_hip_link, child back_right_knee_link, origin xyz=0 -0.02 -0.3 rpy=0 0 0, axis 0 1 0, limit lower=-3.14 upper=3.14 effort=1.0 velocity=1.0
- added joint front_left_abad_joint: type revolute, parent base_link, child front_left_abad_link, origin xyz=0.1 0.1 0 rpy=0 0 0, axis 1 0 0, limit lower=-1.5 upper=1.5 effort=1.0 velocity=1.0
- added joint front_left_hip_joint: type revolute, parent front_left_abad_link, child front_left_hip_link, origin xyz=0 0.02 0 rpy=0 0 0, axis 0 1 0, limit lower=-3.14 upper=3.14 effort=1.0 velocity=1.0
- added joint front_left_knee_joint: type revolute, parent front_left_hip_link, child front_left_knee_link, origin xyz=0 0.02 -0.3 rpy=0 0 0, axis 0 1 0, limit lower=-3.14 upper=3.14 effort=1.0 velocity=1.0
- added joint front_right_abad_joint: type revolute, parent base_link, child front_right_abad_link, origin xyz=0.1 -0.1 0 rpy=0 0 0, axis 1 0 0, limit lower=-1.5 upper=1.5 effort=1.0 velocity=1.0
- added joint front_right_hip_joint: type revolute, parent front_right_abad_link, child front_right_hip_link, origin xyz=0 -0.02 0 rpy=0 0 0, axis 0 1 0, limit lower=-3.14 upper=3.14 effort=1.0 velocity=1.0
- added joint front_right_knee_joint: type revolute, parent front_right_hip_link, child front_right_knee_link, origin xyz=0 -0.02 -0.3 rpy=0 0 0, axis 0 1 0, limit lower=-3.14 upper=3.14 effort=1.0 velocity=1.0

Commit message: 이제 걸음! urdf 파일 수정
아직 걸음 모션 개선 필요...

File: robot_model.urdf (robot description, URDF)
Before this commit: robot quadruped_robot, 13 links, 12 joints
Links:
- link back_left_abad_link: mass 0.3 -> 0.5
- link back_left_hip_link: mass 0.5 -> 0.7; geometry collision cylinder length=0.2 radius=0.03; visual cylinder length=0.2 radius=0.03
- link back_left_knee_link: mass 0.3 -> 0.4; geometry collision cylinder length=0.2 radius=0.03; visual cylinder length=0.2 radius=0.03
- link back_right_abad_link: mass 0.3 -> 0.5
- link back_right_hip_link: mass 0.5 -> 0.7; geometry collision cylinder length=0.2 radius=0.03; visual cylinder length=0.2 radius=0.03
- link back_right_knee_link: mass 0.3 -> 0.4; geometry collision cylinder length=0.2 radius=0.03; visual cylinder length=0.2 radius=0.03
- link base_link: mass 1.0 -> 3.0; geometry collision box size=0.3 0.3 0.1; visual box size=0.4 0.2 0.1
- link front_left_abad_link: mass 0.3 -> 0.5
- link front_left_hip_link: mass 0.5 -> 0.7; geometry collision cylinder length=0.2 radius=0.03; visual cylinder length=0.2 radius=0.03
- link front_left_knee_link: mass 0.3 -> 0.4; geometry collision cylinder length=0.2 radius=0.03; visual cylinder length=0.2 radius=0.03
- link front_right_abad_link: mass 0.3 -> 0.5
- link front_right_hip_link: mass 0.5 -> 0.7; geometry collision cylinder length=0.2 radius=0.03; visual cylinder length=0.2 radius=0.03
- link front_right_knee_link: mass 0.3 -> 0.4; geometry collision cylinder length=0.2 radius=0.03; visual cylinder length=0.2 radius=0.03
Joints:
- joint back_left_abad_joint: origin xyz=-0.1 0.1 0 rpy=0 0 0 -> xyz=-0.13 0.1 0 rpy=0 0 0
- joint back_left_knee_joint: origin xyz=0 0.02 -0.3 rpy=0 0 0 -> xyz=0 0.02 -0.2 rpy=0 0 0
- joint back_right_abad_joint: origin xyz=-0.1 -0.1 0 rpy=0 0 0 -> xyz=-0.13 -0.1 0 rpy=0 0 0
- joint back_right_knee_joint: origin xyz=0 -0.02 -0.3 rpy=0 0 0 -> xyz=0 -0.02 -0.2 rpy=0 0 0
- joint front_left_abad_joint: origin xyz=0.1 0.1 0 rpy=0 0 0 -> xyz=0.15 0.1 0 rpy=0 0 0
- joint front_left_knee_joint: origin xyz=0 0.02 -0.3 rpy=0 0 0 -> xyz=0 0.02 -0.2 rpy=0 0 0
- joint front_right_abad_joint: origin xyz=0.1 -0.1 0 rpy=0 0 0 -> xyz=0.15 -0.1 0 rpy=0 0 0
- joint front_right_knee_joint: origin xyz=0 -0.02 -0.3 rpy=0 0 0 -> xyz=0 -0.02 -0.2 rpy=0 0 0
